File: electronics/MACK10_Controller/MACK10_Controller.kicad_sch (KiCad schematic)
At the start: 0 parts

Commit message: Added KiCad and Electronics Files
Parts:
- added M1: Stepper_Motor_bipolar, symbol Motor:Stepper_Motor_bipolar
- added U1: U1 ESP32_DEVKIT_30P, MACK10:ESP32_DEVKIT_30PIN, symbol MACK10:ESP32_DEVKIT_30P
- added U2: HX711, MACK10:HX711_MODULE, symbol MACK10:HX711_MODULE
- added U3: TMC2208, MACK10:TMC2208_STEPSTICK, symbol MACK10:TMC2208_STEPSTICK
- added U4: LOAD CELL, symbol MACK10:LOAD_CELL_4P
Connections:
- new net: M1.1, U3.12 (1A)
- new net: M1.2 (-), U3.11 (1B)
- new net: M1.3, U3.13 (2A)
- new net: M1.4, U3.14 (2B)
- new net 3V3: U1.1 (3V3), U2.10 (VCC), U3.15 (VIO)
- new net DIR: U1.10 (D19), U3.8 (DIR)
- new net ENABLE: U1.8 (D5), U3.1 (EN)
- new net GND: U1.2 (GND), U2.7 (GND), U3.10 (GND), U3.16 (GND)
- new net HX711_DT: U1.11 (D21), U2.8 (DT)
- new net HX711_SCK: U1.14 (D22), U2.9 (SCK)
- new net LOAD_A+: U2.3 (A-), U4.3 (Pin_3)
- new net LOAD_A-: U2.4 (A+), U4.4 (Pin_4)
- new net LOAD_E+: U2.1 (E+), U4.1 (Pin_1)
- new net LOAD_E-: U2.2 (E-), U4.2 (Pin_2)
- new net STEP: U1.9 (D18), U3.7 (STEP)
Other:
- title: (none) -> MACK-10 Controller

Commit message: Initial PCB Layout
Parts:
- added C1: 100uF 35V, Capacitor_THT:CP_Radial_D8.0mm_P3.50mm, symbol Device:C_Polarized
- added C2: 100nF 50V, Capacitor_THT:C_Disc_D5.0mm_W2.5mm_P5.00mm, symbol Device:C
- added D1: LED, LED_THT:LED_D5.0mm, symbol Device:LED
- added F1: 2A Fuse, Fuse:Fuseholder_Blade_Mini_Keystone_3568, symbol Device:Fuse
- added J1: Stepper Motor, Connector_PinHeader_2.54mm:PinHeader_1x04_P2.54mm_Vertical, symbol Connector_Generic:Conn_01x04
- added J10: POWER SWITCH, Connector_PinHeader_2.54mm:PinHeader_1x02_P2.54mm_Vertical, symbol Connector_Generic:Conn_01x02
- added J2: TMC2208, Connector_PinHeader_2.54mm:PinHeader_1x04_P2.54mm_Vertical, symbol Connector_Generic:Conn_01x04
- added J4: 24V POWER INPUT, Connector_PinHeader_2.54mm:PinHeader_1x04_P2.54mm_Vertical, symbol Connector_Generic:Conn_01x02
- added J5, J6: SSD1306, Connector_PinHeader_2.54mm:PinHeader_1x04_P2.54mm_Vertical, symbol Connector_Generic:Conn_01x04
- added J7: E_STOP, Connector_PinHeader_2.54mm:PinHeader_1x04_P2.54mm_Vertical, symbol Connector_Generic:Conn_01x02
- added J8: LIMIT_TOP, Connector_PinHeader_2.54mm:PinHeader_1x04_P2.54mm_Vertical, symbol Connector_Generic:Conn_01x02
- added J9: LIMIT_BOTTOM, Connector_PinHeader_2.54mm:PinHeader_1x04_P2.54mm_Vertical, symbol Connector_Generic:Conn_01x02
- added R1: 330R, Resistor_THT:R_Axial_DIN0207_L6.3mm_D2.5mm_P10.16mm_Horizontal, symbol Device:R
- added R2, R3: 10k, Resistor_THT:R_Axial_DIN0207_L6.3mm_D2.5mm_P10.16mm_Horizontal, symbol Device:R
- added SW1: SW_UP, Button_Switch_THT:SW_PUSH_6mm, symbol Switch:SW_Push
- added SW2: SW_DOWN, Button_Switch_THT:SW_PUSH_6mm, symbol Switch:SW_Push
- added SW3: SW_SELECT, Button_Switch_THT:SW_PUSH_6mm, symbol Switch:SW_Push
- added SW4: SW_BACK, Button_Switch_THT:SW_PUSH_6mm, symbol Switch:SW_Push
- added U4: LM2596 Buck Converter, MACK10:LM2596_BUCK_CONVERTER, symbol MACK10:LM2596_MODULE
- J3: renamed from U4; value LOAD CELL -> Load Cell; footprint (none) -> Connector_PinHeader_2.54mm:PinHeader_1x04_P2.54mm_Vertical
Connections:
- net 3V3: now also J5.2 (Pin_2)
- net GND: now also U1.17 (GND), C1.2, C2.2, D1.1 (K), J4.2 (Pin_2), J5.1 (Pin_1), J6.1 (Pin_1), J7.2 (Pin_2), J8.2 (Pin_2), J9.2 (Pin_2), SW1.2, SW2.2, SW3.2, SW4.2, U4.2 (IN-), U4.4 (OUT-)
- net +5V: now reaches U1.16 (VIN)
- net +5V: now also U4.3 (OUT+)
- net UP: now reaches U1.18 (D13)
- net UP: now also SW1.1
- net DOWN: now reaches U1.19 (D12)
- net DOWN: now also SW2.1
- net SELECT: now reaches U1.20 (D14)
- net SELECT: now also SW3.1
- net BACK: now reaches U1.21 (D27)
- net BACK: now also SW4.1
- net ESP32 D25: now reaches U1.23 (D25)
- net ESP32 D25: now also J7.1 (Pin_1)
- net ESP32 D33: now reaches U1.24 (D33)
- net ESP32 D33: now also J5.3 (Pin_3)
- net ESP32 D32: now reaches U1.25 (D32)
- net ESP32 D32: now also J5.4 (Pin_4)
- net ESP32 D35: now reaches U1.26 (D35)
- net ESP32 D35: now also R2.1
- net ESP32 D34: now reaches U1.27 (D34)
- net ESP32 D34: now also R3.1
- net ESP32 D4: now reaches U1.5 (D4)
- net ESP32 D4: now also R1.1
- net at U3.12 (1A): now also J1.2 (Pin_2); no longer M1.1
- net at U3.11 (1B): now also J1.1 (Pin_1); no longer M1.2 (-)
- net at U3.13 (2A): now also J1.3 (Pin_3); no longer M1.3
- net at U3.14 (2B): now also J1.4 (Pin_4); no longer M1.4
- net +24V: now reaches U3.9 (VMOT)
- net +24V: now also C1.1, C2.1, J10.1 (Pin_1), U4.1 (IN+)
- new net: J8.1 (Pin_1), R2.2
- new net: F1.2, J10.2 (Pin_2)
- new net: J9.1 (Pin_1), R3.2
- new net: D1.2 (A), R1.2
- new net 24V INPUT: F1.1, J4.1 (Pin_1)
- new net PIN 1: J2.1 (Pin_1), M1.1
- new net PIN 2: J2.2 (Pin_2), M1.2 (-)
- new net PIN 3: J2.3 (Pin_3), M1.3
- new net PIN 4: J2.4 (Pin_4), M1.4
- new net SCL: J6.3 (Pin_3)
- new net SDA: J6.4 (Pin_4)
- new net VCC: J6.2 (Pin_2)
- no-connect marks 0 -> 21
Other:
- moved on the sheet: J3, M1, U1, U2, U3

Commit message: Update PCB Layout
Parts:
- removed J2: TMC2208, Connector_PinHeader_2.54mm:PinHeader_1x04_P2.54mm_Vertical, symbol Connector_Generic:Conn_01x04
- removed J5: SSD1306, Connector_PinHeader_2.54mm:PinHeader_1x04_P2.54mm_Vertical, symbol Connector_Generic:Conn_01x04
- removed M1: Stepper_Motor_bipolar, symbol Motor:Stepper_Motor_bipolar
- removed SW1: SW_UP, Button_Switch_THT:SW_PUSH_6mm, symbol Switch:SW_Push
- removed SW2: SW_DOWN, Button_Switch_THT:SW_PUSH_6mm, symbol Switch:SW_Push
- removed SW3: SW_SELECT, Button_Switch_THT:SW_PUSH_6mm, symbol Switch:SW_Push
- removed SW4: SW_BACK, Button_Switch_THT:SW_PUSH_6mm, symbol Switch:SW_Push
- added D2: STATUS LED, LED_SMD:LED_0805_2012Metric_Pad1.15x1.40mm_HandSolder, symbol Device:LED
- added J6: INPUT, Connector_JST:JST_XH_B6B-XH-A_1x06_P2.50mm_Vertical, symbol Connector_Generic:Conn_01x06
- added R4: 1k, Resistor_THT:R_Axial_DIN0207_L6.3mm_D2.5mm_P10.16mm_Horizontal, symbol Device:R
- D1: value LED -> POWER LED; footprint LED_THT:LED_D5.0mm -> LED_SMD:LED_0805_2012Metric_Pad1.15x1.40mm_HandSolder
- J1, J3: footprint Connector_PinHeader_2.54mm:PinHeader_1x04_P2.54mm_Vertical -> Connector_JST:JST_XH_B4B-XH-A_1x04_P2.50mm_Vertical
- J4, J7, J8, J9: footprint Connector_PinHeader_2.54mm:PinHeader_1x04_P2.54mm_Vertical -> Connector_JST:JST_XH_B2B-XH-A_1x02_P2.50mm_Vertical
- J5: renamed from J6; footprint Connector_PinHeader_2.54mm:PinHeader_1x04_P2.54mm_Vertical -> Connector_JST:JST_XH_B4B-XH-A_1x04_P2.50mm_Vertical
- R1: value 330R -> 1k
Connections:
- net SCL is gone; now on net ESP32 D33: J5.3 (SCL)
- net SDA is gone; now on net ESP32 D32: J5.4 (SDA)
- net VCC is gone; now on net 3V3: J5.2 (VCC)
- net 3V3: now also R1.1
- net BACK: now also J6.5 (Pin_5)
- net DOWN: now also J6.3 (Pin_3)
- net ESP32 D4: now also R4.1; no longer R1.1
- net GND: now also D2.1 (K), J6.1 (Pin_1)
- net SELECT: now also J6.4 (Pin_4)
- net UP: now also J6.2 (Pin_2)
- new net: D2.2 (A), R4.2
- no-connect marks 21 -> 19
Other:
- moved on the sheet: F1, J10, J4, J8, J9, R2, R3, U4

Commit message: Various PCB Updates
Parts:
- added 24VI1: TP5, TestPoint:TestPoint_Pad_2.0x2.0mm, symbol Connector:TestPoint
- added 3V3: TP1, TestPoint:TestPoint_Pad_2.0x2.0mm, symbol Connector:TestPoint
- added 5VO1: TP3, TestPoint:TestPoint_Pad_2.0x2.0mm, symbol Connector:TestPoint
- added EN1: TP7, TestPoint:TestPoint_Pad_2.0x2.0mm, symbol Connector:TestPoint
- added GND1: TP4, TestPoint:TestPoint_Pad_2.0x2.0mm, symbol Connector:TestPoint
- added HXDT1: TP2, TestPoint:TestPoint_Pad_2.0x2.0mm, symbol Connector:TestPoint
- added HXSCK1: TP6, TestPoint:TestPoint_Pad_2.0x2.0mm, symbol Connector:TestPoint
- added SDIR1: TP9, TestPoint:TestPoint_Pad_2.0x2.0mm, symbol Connector:TestPoint
- added STEP1: TP8, TestPoint:TestPoint_Pad_2.0x2.0mm, symbol Connector:TestPoint
Connections:
- net +24V: now also 24VI1.1
- net +5V: now also 5VO1.1
- net 3V3: now also 3V3.1
- net DIR: now also SDIR1.1
- net ENABLE: now also EN1.1
- net GND: now also GND1.1
- net HX711_DT: now also HXDT1.1
- net HX711_SCK: now also HXSCK1.1
- net STEP: now also STEP1.1
Other:
- moved on the sheet: C1, C2, J1, J3, U2, U3, U4

Commit message: Various PSB and Schematic Updates
Parts:
- D1: value POWER LED -> POWER
- D2: value STATUS LED -> STATUS
- J10: value POWER SWITCH -> I/O
- J4: value 24V POWER INPUT -> 24V IN
- J8: value LIMIT_TOP -> LIM_TOP
- J9: value LIMIT_BOTTOM -> LIM_BOT
- renumbered 24VI1 to 24VIN1, 5VO1 to 5VOUT1
Changed lines of the file:
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@@
 			)
 		)
-		(property "Value" "LIMIT_BOTTOM"
+		(property "Value" "LIM_BOT"
 			(at 260.35 111.7599 0)
 			(show_name no)
@@
 		(dnp no)
 		(fields_autoplaced yes)
-		(property "Reference" "5VO1"
+		(property "Reference" "5VOUT1"
 			(at 273.05 140.2079 0)
 			(show_name no)
@@
 			(project "MACK10_Controller"
 				(path "/ab42f44a-5ab9-4a28-b026-e4608900329e"
-					(reference "5VO1")
+					(reference "5VOUT1")
 					(unit 1)
 				)
@@
 			)
 		)
-		(property "Value" "LIMIT_TOP"
+		(property "Value" "LIM_TOP"
 			(at 260.35 100.3299 0)
 			(show_name no)
@@
 		(dnp no)
 		(fields_autoplaced yes)
-		(property "Reference" "24VI1"
+		(property "Reference" "24VIN1"
 			(at 240.03 138.9379 0)
 			(show_name no)
@@
 			(project "MACK10_Controller"
 				(path "/ab42f44a-5ab9-4a28-b026-e4608900329e"
-					(reference "24VI1")
+					(reference "24VIN1")
 					(unit 1)
 				)
@@
 			)
 		)
-		(property "Value" "24V POWER INPUT"
+		(property "Value" "24V IN"
 			(at 200.66 130.8099 0)
 			(show_name no)
@@
 			)
 		)
-		(property "Value" "POWER SWITCH"
+		(property "Value" "I/O"
 			(at 256.54 134.6199 90)
 			(show_name no)
@@
 			)
 		)
-		(property "Value" "STATUS LED"
+		(property "Value" "STATUS"
 			(at 249.2375 82.55 0)
 			(show_name no)
@@
 			)
 		)
-		(property "Value" "POWER LED"
+		(property "Value" "POWER"
 			(at 249.2375 71.12 0)
 			(show_name no)

Commit message: Add Todo and various PCB updates
Parts:
- added JP1: FUSE_BYPASS, Jumper:SolderJumper-2_P1.3mm_Open_Pad1.0x1.5mm, symbol Jumper:Jumper_2_Open
- C1: footprint Capacitor_THT:CP_Radial_D8.0mm_P3.50mm -> Capacitor_SMD:CP_Elec_6.3x5.4
- C2: footprint Capacitor_THT:C_Disc_D5.0mm_W2.5mm_P5.00mm -> Capacitor_SMD:C_0603_1608Metric
- F1: footprint Fuse:Fuseholder_Blade_Mini_Keystone_3568 -> Connector_JST:JST_XH_B2B-XH-A_1x02_P2.50mm_Vertical; symbol Device:Fuse -> Connector_Generic:Conn_01x02
- J10: footprint Connector_PinHeader_2.54mm:PinHeader_1x02_P2.54mm_Vertical -> Connector_JST:JST_XH_B2B-XH-A_1x02_P2.50mm_Vertical
- R1, R2, R3, R4: footprint Resistor_THT:R_Axial_DIN0207_L6.3mm_D2.5mm_P10.16mm_Horizontal -> Resistor_SMD:R_0603_1608Metric
Connections:
- net 24V INPUT: now also JP1.1 (A)
- net at F1.2 (Pin_2), J10.2 (Pin_2): now also JP1.2 (B)
Other:
- moved on the sheet: J10, J4, J8, J9, R2, R3

Commit message: Various PCB and Schematic Updates
Parts:
- J1: value Stepper Motor -> Motor
- J4: footprint Connector_JST:JST_XH_B2B-XH-A_1x02_P2.50mm_Vertical -> Connector_BarrelJack:BarrelJack_CUI_PJ-102AH_Horizontal
- TP1: renamed from 3V3; value TP1 -> 3V3
- TP2: renamed from HXDT1; value TP2 -> HXDT
- TP3: renamed from 5VOUT1; value TP3 -> 5VOUT
- TP4: renamed from GND1; value TP4 -> GND
- TP5: renamed from 24VIN1; value TP5 -> 24VIN
- TP6: renamed from HXSCK1; value TP6 -> HXSCK
- TP7: renamed from EN1; value TP7 -> EN
- TP8: renamed from STEP1; value TP8 -> STEP
- TP9: renamed from SDIR1; value TP9 -> SDIR
Connections:
- net 24V INPUT: no longer names the net of F1.1 (Pin_1), J4.1 (Pin_1), JP1.1 (A)
Other:
- moved on the sheet: F1, J10, J4, JP1

Commit message: PCB Traces Completed - First Run
Parts:
- J4: symbol Connector_Generic:Conn_01x02 -> Connector_Generic:Conn_01x03
- TP5: value 24VIN -> 24V
Connections:
- net +24V: now also J10.2 (Pin_2); no longer J10.1 (Pin_1)
- net 24VIN: now reaches F1.1 (Pin_1), J4.1 (Pin_1), JP1.1 (A)
- net at F1.2 (Pin_2), JP1.2 (B): now also J10.1 (Pin_1); no longer J10.2 (Pin_2)
- no-connect marks 19 -> 9
Other:
- moved on the sheet: F1, J10, JP1
