File: electronics/MACK10_Controller/MACK10_Controller.kicad_sch (KiCad schematic)
At the start: 32 parts, among them J1 Motor, J10 I/O, J3 Load Cell, J4 24V IN, J5 SSD1306, J6 INPUT, J7 E_STOP, J8 LIM_TOP, J9 LIM_BOT, U1 U1 ESP32_DEVKIT_30P, U2 HX711, U3 TMC2208, U4 LM2596 Buck Converter

Commit message: RevA PCB Layout Finalized
Parts:
- C1: footprint Capacitor_SMD:CP_Elec_6.3x5.4 -> Capacitor_SMD:CP_Elec_6.3x7.7
- C2: footprint Capacitor_SMD:C_0603_1608Metric -> Capacitor_SMD:C_0805_2012Metric
- R1, R2, R3, R4: footprint Resistor_SMD:R_0603_1608Metric -> Resistor_SMD:R_0805_2012Metric
Connections:
- net 3V3: now also R2.1, R3.1
- net DOWN: now also U1.22 (D26); no longer U1.19 (D12)
- net ESP32 D34: now also J9.1 (Pin_1), R3.2; no longer R3.1
- net ESP32 D35: now also J8.1 (Pin_1), R2.2; no longer R2.1
- net GND: now also J4.3 (Pin_3); no longer J4.2 (Pin_2)
- net LOAD_A+: now also U2.4 (A+); no longer U2.3 (A-)
- net LOAD_A-: now also U2.3 (A-); no longer U2.4 (A+)
Other:
- moved on the sheet: R2, R3
