File: electronics/MACK10_Controller/MACK10_Controller.kicad_pcb (KiCad board)
At the start: 2 copper layers, 25 parts, among them J1 Stepper Motor, J10 POWER SWITCH, J2 TMC2208, J3 Load Cell, J4 24V POWER INPUT, J5 SSD1306, J6 SSD1306, J7 E_STOP, J8 LIMIT_TOP, J9 LIMIT_BOTTOM, SW1 SW_UP, SW2 SW_DOWN, SW3 SW_SELECT, SW4 SW_BACK, U1 U1 ESP32_DEVKIT_30P, U2 HX711, U3 TMC2208, U4 LM2596 Buck Converter

Commit message: Update PCB Layout
Parts:
- removed J2: TMC2208, Connector_PinHeader_2.54mm:PinHeader_1x04_P2.54mm_Vertical
- removed the J5 at (74.2, 50.3)
- removed SW1: SW_UP, Button_Switch_THT:SW_PUSH_6mm
- removed SW2: SW_DOWN, Button_Switch_THT:SW_PUSH_6mm
- removed SW3: SW_SELECT, Button_Switch_THT:SW_PUSH_6mm
- removed SW4: SW_BACK, Button_Switch_THT:SW_PUSH_6mm
- added D2: STATUS LED, LED_SMD:LED_0805_2012Metric_Pad1.15x1.40mm_HandSolder, F.Cu at (73.5, 95.5)
- added J6: INPUT, Connector_JST:JST_XH_B6B-XH-A_1x06_P2.50mm_Vertical, F.Cu at (36.2, 106.5)
- added R4: 1k, Resistor_THT:R_Axial_DIN0207_L6.3mm_D2.5mm_P10.16mm_Horizontal, F.Cu at (48.7, 107.0)
- D1: value LED -> POWER LED; footprint LED_THT:LED_D5.0mm -> LED_SMD:LED_0805_2012Metric_Pad1.15x1.40mm_HandSolder
- J1, J3: footprint Connector_PinHeader_2.54mm:PinHeader_1x04_P2.54mm_Vertical -> Connector_JST:JST_XH_B4B-XH-A_1x04_P2.50mm_Vertical
- J4, J7, J8, J9: footprint Connector_PinHeader_2.54mm:PinHeader_1x04_P2.54mm_Vertical -> Connector_JST:JST_XH_B2B-XH-A_1x02_P2.50mm_Vertical
- J5: renamed from J6; footprint Connector_PinHeader_2.54mm:PinHeader_1x04_P2.54mm_Vertical -> Connector_JST:JST_XH_B4B-XH-A_1x04_P2.50mm_Vertical
- R1: value 330R -> 1k
- moved J9 83.0 mm to (24.0, 97.0)
- moved J8 74.2 mm to (24.0, 88.0)
- moved J7 66.0 mm to (24.0, 79.0)
- moved U3 62.5 mm to (91.6, 52.0)
- moved F1 57.2 mm to (92.5, 103.5)
- moved J5 56.9 mm to (36.2, 88.0)
- moved J4 53.8 mm to (72.0, 104.0)
- moved C2 49.5 mm to (103.5, 96.0), turned to 90 degrees
- moved J1 46.0 mm to (92.1, 78.5)
- moved J3 40.8 mm to (36.0, 79.0)
- moved C1 35.7 mm to (92.0, 93.5)
- moved J10 12.3 mm to (64.8, 103.7)
- moved R1 12.2 mm to (48.9, 95.0)
- moved R2 12.2 mm to (48.9, 99.0)
- moved R3 12.2 mm to (48.9, 103.1)
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Connections:
- J5 pad 2: /VCC -> /3V3
- J5 pad 3: /SCL -> /ESP32 D33
- J5 pad 4: /SDA -> /ESP32 D32
- R1 pad 1: /ESP32 D4 -> /3V3
Other:
- board text added: "3V3"
- board text added: "GND"
- board text added: "SCL"
- board text added: "SDA"

Commit message: Minor PCB Updates
Other:
- board outline added: 93.5 x 100.5 mm
Changed lines of the file:
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@@
 			(outputformat 1)
 			(mirror no)
-			(drillshape 1)
+			(drillshape 0)
 			(scaleselection 1)
-			(outputdirectory "")
+			(outputdirectory "../../../../../../../../../../../Downloads/Gerbers/")
 		)
 	)
@@
 		)
 	)
+	(gr_rect
+		(start 17 13.5)
+		(end 110.5 114)
+		(stroke
+			(width 0.05)
+			(type default)
+		)
+		(fill no)
+		(layer "Edge.Cuts")
+	)
 	(gr_text "GND\n"

Commit message: Various PCB Updates
Parts:
- added 24VI1: TP5, TestPoint:TestPoint_Pad_2.0x2.0mm, F.Cu at (109.5, 30.5)
- added 3V3: TP1, TestPoint:TestPoint_Pad_2.0x2.0mm, F.Cu at (109.5, 18.5)
- added 5VO1: TP3, TestPoint:TestPoint_Pad_2.0x2.0mm, F.Cu at (109.5, 24.5)
- added EN1: TP7, TestPoint:TestPoint_Pad_2.0x2.0mm, F.Cu at (109.5, 36.5)
- added GND1: TP4, TestPoint:TestPoint_Pad_2.0x2.0mm, F.Cu at (109.5, 27.5)
- added HXDT1: TP2, TestPoint:TestPoint_Pad_2.0x2.0mm, F.Cu at (109.5, 21.5)
- added HXSCK1: TP6, TestPoint:TestPoint_Pad_2.0x2.0mm, F.Cu at (109.5, 33.5)
- added SDIR1: TP9, TestPoint:TestPoint_Pad_2.0x2.0mm, F.Cu at (109.5, 42.5)
- added STEP1: TP8, TestPoint:TestPoint_Pad_2.0x2.0mm, F.Cu at (109.5, 39.5)
Other:
- board size 93.5 x 100.5 mm -> 97.4 x 100.5 mm

Commit message: Various PSB and Schematic Updates
Parts:
- D1: value POWER LED -> POWER
- D2: value STATUS LED -> STATUS
- J10: value POWER SWITCH -> I/O
- J4: value 24V POWER INPUT -> 24V IN
- J8: value LIMIT_TOP -> LIM_TOP
- J9: value LIMIT_BOTTOM -> LIM_BOT
- moved GND1 16.4 mm to (109.5, 44.0)
- moved EN1 3.05 mm to (109.5, 33.5)
- moved STEP1 3.05 mm to (109.5, 36.5)
- moved HXSCK1 3.05 mm to (109.5, 30.5)
- moved 24VIN1 3.05 mm to (109.5, 27.5)
- moved SDIR1 3.05 mm to (109.5, 39.5)
- renumbered 24VI1 to 24VIN1, 5VO1 to 5VOUT1
Other:
- board text added: "ESP32"

Commit message: Add Todo and various PCB updates
Parts:
- added JP1: FUSE_BYPASS, Jumper:SolderJumper-2_P1.3mm_Open_Pad1.0x1.5mm, F.Cu at (95.0, 90.8)
- added REF**: MountingHole_3.2mm_M3, MountingHole:MountingHole_3.2mm_M3, F.Cu at (25.0, 25.0)
- added REF**: MountingHole_3.2mm_M3, MountingHole:MountingHole_3.2mm_M3, F.Cu at (105.0, 100.0)
- added REF**: MountingHole_3.2mm_M3, MountingHole:MountingHole_3.2mm_M3, F.Cu at (105.0, 25.0)
- added REF**: MountingHole_3.2mm_M3, MountingHole:MountingHole_3.2mm_M3, F.Cu at (24.5, 100.0)
- added TP4: GND, TestPoint:TestPoint_Pad_2.0x2.0mm, F.Cu at (28.0, 89.0)
- C1: footprint Capacitor_THT:CP_Radial_D8.0mm_P3.50mm -> Capacitor_SMD:CP_Elec_6.3x5.4
- C2: footprint Capacitor_THT:C_Disc_D5.0mm_W2.5mm_P5.00mm -> Capacitor_SMD:C_0603_1608Metric
- F1: footprint Fuse:Fuseholder_Blade_Mini_Keystone_3568 -> Connector_JST:JST_XH_B2B-XH-A_1x02_P2.50mm_Vertical
- J10: footprint Connector_PinHeader_2.54mm:PinHeader_1x02_P2.54mm_Vertical -> Connector_JST:JST_XH_B2B-XH-A_1x02_P2.50mm_Vertical
- R1, R2, R3, R4: footprint Resistor_THT:R_Axial_DIN0207_L6.3mm_D2.5mm_P10.16mm_Horizontal -> Resistor_SMD:R_0603_1608Metric
- TP1: renamed from 3V3; value TP1 -> 3V3
- TP2: renamed from HXDT1; value TP2 -> HXDT
- TP3: renamed from 5VOUT1; value TP3 -> 5VOUT
- TP4: renamed from GND1; value TP4 -> GND
- TP5: renamed from 24VIN1; value TP5 -> 24VIN
- TP6: renamed from HXSCK1; value TP6 -> HXSCK
- TP7: renamed from EN1; value TP7 -> EN
- TP8: renamed from STEP1; value TP8 -> STEP
- TP9: renamed from SDIR1; value TP9 -> SDIR
- moved TP1 101.5 mm to (28.0, 79.0)
- moved TP5 99.8 mm to (28.0, 85.0)
- moved TP3 99.8 mm to (28.0, 82.0)
- moved TP2 68.1 mm to (73.8, 79.5), turned to 90 degrees
- moved TP6 59.0 mm to (76.7, 79.5), turned to 90 degrees
- moved TP7 54.8 mm to (79.7, 79.5), turned to 90 degrees
- moved TP8 50.6 mm to (82.8, 79.5), turned to 90 degrees
- moved C1 49.2 mm to (43.0, 98.3)
- moved TP9 46.5 mm to (85.8, 79.5), turned to 90 degrees
- moved R4 43.2 mm to (90.9, 97.5)
- moved J7 42.9 mm to (65.8, 89.0)
- moved TP4 40.4 mm to (90.2, 79.5), turned to 90 degrees
- moved R3 38.9 mm to (87.4, 97.5)
- moved R2 35.0 mm to (83.9, 97.5)
- moved F1 32.0 mm to (61.0, 98.0)
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Other:
- board outline removed
- board text removed: "3V3"
- board text removed: "GND"
- board text removed: "SCL"
- board text removed: "SDA"

Commit message: Various PCB and Schematic Updates
Parts:
- removed the TP4 at (28.0, 89.0)
- removed the TP4 at (90.2, 79.5)
- added TP4: GND, TestPoint:TestPoint_Pad_2.0x2.0mm, F.Cu at (30.0, 102.8)
- J1: value Stepper Motor -> Motor
- J4: footprint Connector_JST:JST_XH_B2B-XH-A_1x02_P2.50mm_Vertical -> Connector_BarrelJack:BarrelJack_CUI_PJ-102AH_Horizontal
- moved R4 80.1 mm to (45.2, 31.7), turned to 90 degrees
- moved R3 75.3 mm to (45.2, 35.2), turned to 90 degrees
- moved D2 72.3 mm to (54.0, 36.8), turned to 90 degrees
- moved R2 70.4 mm to (45.2, 38.7), turned to 90 degrees
- moved D1 67.9 mm to (56.2, 36.8), turned to 90 degrees
- moved R1 65.6 mm to (45.2, 42.2), turned to 90 degrees
- moved J4 65.3 mm to (85.6, 34.6), turned to 90 degrees
- moved J9 57.0 mm to (89.8, 54.4)
- moved TP9 57.0 mm to (33.8, 102.8), turned to -90 degrees
- moved J8 54.8 mm to (89.9, 47.2)
- moved TP8 51.5 mm to (36.8, 102.8), turned to -90 degrees
- moved J10 48.2 mm to (90.0, 68.4)
- moved C1 47.0 mm to (87.9, 84.0)
- moved TP7 46.3 mm to (39.8, 102.8), turned to -90 degrees
- moved J6 42.4 mm to (75.9, 91.8), turned to 0 degrees
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Connections:
- net /24V INPUT renamed Net-(F1-Pin_1)

Commit message: PCB Traces Completed - First Run
Parts:
- TP5: value 24VIN -> 24V
- moved TP4 0.35 mm to (30.4, 102.8), turned to 0 degrees
- moved TP1 0.23 mm to (55.0, 102.8)
- moved TP3 0.13 mm to (51.9, 102.8)
- moved TP5 0.08 mm to (48.9, 102.8)
Connections:
- net Net-(F1-Pin_1) renamed /24VIN
- J10 pad 1: /+24V -> Net-(F1-Pin_2)
- J10 pad 2: Net-(F1-Pin_2) -> /+24V
- J4 pad 3: (no net) -> unconnected-(J4-Pin_3-Pad3)
- TP4 pad 1: (no net) -> /GND
Routing:
- net /GND: track 0.00 -> 367.3 mm, vias 0 -> 4
- net /3V3: track 0.00 -> 271.6 mm, vias 0 -> 4
- net /+24V: track 0.00 -> 182.9 mm
- net Net-(J9-Pin_1): track 0.00 -> 167.4 mm
- net /ESP32 D32: track 0.00 -> 147.5 mm
- net /DIR: track 0.00 -> 137.2 mm, vias 0 -> 1
- net /ESP32 D33: track 0.00 -> 134.6 mm
- net Net-(J8-Pin_1): track 0.00 -> 120.4 mm, vias 0 -> 3
- net /ENABLE: track 0.00 -> 112.6 mm, vias 0 -> 2
- net /STEP: track 0.00 -> 112.1 mm, vias 0 -> 2
- net /+5V: track 0.00 -> 105.2 mm
- net /UP: track 0.00 -> 88.8 mm, vias 0 -> 1
- net /HX711_DT: track 0.00 -> 87.0 mm, vias 0 -> 2
- net /DOWN: track 0.00 -> 84.3 mm
- net /HX711_SCK: track 0.00 -> 78.6 mm, vias 0 -> 3
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
Commit message: Various PCB Updates
Parts:
- Mount 1: renamed from REF**
- Mount 2: renamed from REF**
- Mount 3: renamed from REF**
- Mount 4: renamed from REF**
- moved TP5 77.6 mm to (97.2, 42.0), turned to 90 degrees
Routing:
- net /GND: track 367.3 -> 281.0 mm, vias 4 -> 16
- net /ESP32 D32: track 147.5 -> 96.9 mm, vias 0 -> 2
- net /+24V: track 182.9 -> 139.1 mm, vias 0 -> 1
- net Net-(J8-Pin_1): track 120.4 -> 93.2 mm, vias 3 -> 5
- net /HX711_SCK: track 78.6 -> 60.6 mm, vias 3 -> 2
- net /HX711_DT: track 87.0 -> 69.2 mm, vias 2 -> 1
- net /ESP32 D4: track 35.1 -> 26.4 mm
- net /3V3: track 271.6 -> 277.6 mm
- net /LOAD_E+: track 52.1 -> 46.9 mm
- net /LOAD_E-: track 52.7 -> 49.0 mm
- net /+5V: track 105.2 -> 103.6 mm
- net Net-(J9-Pin_1): track 167.4 -> 166.2 mm
- net /UP: track 88.8 -> 89.1 mm, vias 1 -> 0
- added copper zone on B.Cu, net /GND
- added copper zone on F.Cu, net /GND
Other:
- board outline added: 80 x 85 mm
