File: electronics/MACK10_Controller/MACK10_Controller.kicad_pcb (KiCad board)
At the start: 2 copper layers, 80 x 85 mm, 36 parts, among them J1 Motor, J10 I/O, J3 Load Cell, J4 24V IN, J5 SSD1306, J6 INPUT, J7 E_STOP, J8 LIM_TOP, J9 LIM_BOT, U1 U1 ESP32_DEVKIT_30P, U2 HX711, U3 TMC2208, U4 LM2596 Buck Converter

Commit message: Finalize V1 PCB Layout
Parts:
- moved U2 2.13 mm to (25.6, 82.8)
- moved TP1 1.36 mm to (54.9, 104.1)
- moved TP2 1.36 mm to (45.7, 104.1)
- moved TP3 1.36 mm to (51.8, 104.1)
- moved TP4 1.36 mm to (30.2, 104.1)
- moved TP6 1.36 mm to (42.6, 104.1)
- moved TP7 1.36 mm to (39.6, 104.1)
- moved TP8 1.36 mm to (36.6, 104.1)
- moved TP9 1.36 mm to (33.6, 104.1)
- moved Mount 2 1.00 mm to (24.5, 101.0)
- moved Mount 4 1.00 mm to (95.0, 101.0)
Routing:
- net /ENABLE: track 112.6 -> 92.9 mm, vias 2 -> 1
- net /STEP: track 112.1 -> 110.1 mm
- net /DIR: track 137.2 -> 135.5 mm
- net /HX711_DT: track 69.2 -> 70.9 mm
- net /ESP32 D33: track 134.2 -> 135.9 mm
- net /3V3: track 277.6 -> 279.3 mm
- net /+5V: track 103.6 -> 105.2 mm
- net /LOAD_E+: track 46.9 -> 46.0 mm
- net /LOAD_E-: track 49.0 -> 48.1 mm
- net /LOAD_A-: track 56.1 -> 55.2 mm
- net /LOAD_A+: track 54.7 -> 53.8 mm
- net Net-(J9-Pin_1): vias 0 -> 2

Commit message: RevA PCB Layout Finalized
Parts:
- C1: footprint Capacitor_SMD:CP_Elec_6.3x5.4 -> Capacitor_SMD:CP_Elec_6.3x7.7
- C2: footprint Capacitor_SMD:C_0603_1608Metric -> Capacitor_SMD:C_0805_2012Metric
- R1, R2, R3, R4: footprint Resistor_SMD:R_0603_1608Metric -> Resistor_SMD:R_0805_2012Metric
- moved C1 2.83 mm to (90.7, 84.1), turned to -90 degrees
- moved C2 1.98 mm to (57.4, 85.8), turned to -90 degrees
- moved R4 0.55 mm to (44.7, 31.5)
- moved R1 0.50 mm to (44.8, 42.2)
- moved R3 0.48 mm to (44.8, 35.1)
- moved R2 0.48 mm to (44.8, 38.6)
Connections:
- J4 pad 2: /GND -> unconnected-(J4-Pin_2-Pad2)
- J4 pad 3: unconnected-(J4-Pin_3-Pad3) -> /GND
- J8 pad 1: Net-(J8-Pin_1) -> /ESP32 D35
- J9 pad 1: Net-(J9-Pin_1) -> /ESP32 D34
- R2 pad 1: /ESP32 D35 -> /3V3
- R2 pad 2: Net-(J8-Pin_1) -> /ESP32 D35
- R3 pad 1: /ESP32 D34 -> /3V3
- R3 pad 2: Net-(J9-Pin_1) -> /ESP32 D34
- U1 pad 19: /DOWN -> unconnected-(U1-D12-Pad19)
- U1 pad 22: unconnected-(U1-D26-Pad22) -> /DOWN
- U2 pad 3: /LOAD_A+ -> /LOAD_A-
- U2 pad 4: /LOAD_A- -> /LOAD_A+
Routing:
- net Net-(J9-Pin_1): track 166.2 -> 0.00 mm, vias 2 -> 0
- net /ESP32 D34: track 28.7 -> 171.3 mm
- net Net-(J8-Pin_1): track 93.2 -> 0.00 mm, vias 5 -> 0
- net /ESP32 D35: track 22.1 -> 103.2 mm, vias 0 -> 3
- net /DOWN: track 84.3 -> 76.0 mm, vias 0 -> 1
- net /LOAD_A-: track 55.2 -> 49.4 mm, vias 1 -> 0
- net /LOAD_A+: track 53.8 -> 48.2 mm
- net /3V3: track 279.3 -> 284.2 mm, vias 4 -> 5
- net /GND: track 281.0 -> 285.4 mm, vias 16 -> 17
- net unconnected-(U1-D26-Pad22): track 2.54 -> 0.00 mm
- net unconnected-(U1-D12-Pad19): track 0.00 -> 2.54 mm
- net /+24V: track 139.1 -> 141.2 mm
- net unconnected-(J4-Pin_2-Pad2): track 0.00 -> 1.13 mm
- net Net-(D2-A): track 11.1 -> 12.1 mm
- net /ESP32 D4: track 26.4 -> 25.7 mm
Other:
- board size 80 x 85 mm -> 80 x 85.7 mm
