File: electronics/MACK10_Controller v2/MACK10_Controller.kicad_pcb (KiCad board)
At the start: 2 copper layers, 80 x 85.7 mm, 36 parts, among them J1 Motor, J10 I/O, J3 Load Cell, J4 24V IN, J5 SSD1306, J6 INPUT, J7 E_STOP, J8 LIM_TOP, J9 LIM_BOT, U1 U1 ESP32_DEVKIT_30P, U2 HX711, U3 TMC2208, U4 LM2596 Buck Converter

Commit message: PCB Updates
Parts:
- JP1: footprint Jumper:SolderJumper-2_P1.3mm_Open_Pad1.0x1.5mm -> Connector_PinHeader_2.54mm:PinHeader_1x02_P2.54mm_Vertical
- moved JP1 13.7 mm to (93.7, 85.2), turned to 180 degrees
- moved C1 2.58 mm to (88.1, 84.2)
