File: electronics/MACK10_Controller v2/MACK10_Controller.kicad_pcb (KiCad board)
At the start: 2 copper layers, 57.3 x 67.1 mm, 61 parts, among them J10 BYP_2, J2 Motor, J3 J_Expansion, J4 I/O, J5 Sensor IDC, J6 Interface IDC, J7 Fan, J8 E_STOP, J9 24V IN, Q1 SS8550, SW1 ENABLE, U1 TMC2208, U2 HX711, U3 XIAO-C6, U4 INA226, U5 PCF8575, U6 MINI360

Commit message: All Checks Passed - V2 Sent for Manufacture
Parts:
- added D3: SS14, Diode_SMD:D_SMA, B.Cu at (49.4, 20.5)
- SW1: value ENABLE -> RESET
Connections:
- U3 pad 14: /+5V -> Net-(D3-K)
Routing:
- net /+5V: track 235.8 -> 246.2 mm, vias 9 -> 11
- net Net-(D3-K): track 0.00 -> 3.92 mm, vias 0 -> 1
- net /IO3: track 39.7 -> 36.2 mm
- net /STATUS: track 42.0 -> 40.4 mm
- net /ENABLE: track 36.8 -> 38.2 mm
- net /SDA: track 168.4 -> 169.3 mm
- net /A+: track 29.5 -> 29.0 mm
- net Net-(U3-EN): vias 6 -> 5
